File: system_design/Georgetown/V0.5.2/EDA/main_board/main_board.kicad_pcb (KiCad board)
At the start: 2 copper layers, 40.6 x 82.6 mm, 36 parts, among them J1 B3B-XH-A_LF__SN_, J2 Conn_01x02_Pin, P1 SD card socket, Q1 MMBT2222A, SW1 SW_Wuerth_450301014042, U1 HX-2S-JH10, U2 DS3231M, U4 BME280_module, U5 KA78M05_TO252

Commit message: BOM and PCB edited for Nano every
Other:
- board text added: "Nano Every"
- board text removed: "Arduino Nano"
Changed lines of the file:
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@@
 		)
 	)
-	(gr_text "Arduino Nano"
+	(gr_text "Nano Every"
 		(at 153.95 127.82 90)
 		(layer "F.SilkS")
